Commit message: new changes

File: zimo_description/urdf/zimo.urdf.xacro (robot description, xacro)
@@ -12,4 +12,10 @@
             </geometry>
         </visual>
+        <collision>
+            <origin xyz="-0.5 -0.5 0" rpy="0 0 0" />
+            <geometry>
+                <mesh filename="package://zimo_description/meshes/zimo/basement.STL" scale="0.01 0.01 0.01" />
+            </geometry>
+        </collision>
     </link>
     <joint name="world_base_link_joint" type="fixed">
@@ -25,4 +31,10 @@
             </geometry>
         </visual>
+        <collision>
+            <origin xyz="-0.39 -0.39 -0.56" rpy="0 0 0" />
+            <geometry>
+                <mesh filename="package://zimo_description/meshes/zimo/base_plate.STL" scale="0.01 0.01 0.01" />
+            </geometry>
+        </collision>
     </link>
     <joint name="joint_1" type="revolute">
@@ -40,4 +52,10 @@
             </geometry>
         </visual>
+        <collision>
+            <origin xyz="0.19 -0.06 -0.08" rpy="0 -${PI/2} ${PI/2}" />
+            <geometry>
+                <mesh filename="package://zimo_description/meshes/zimo/forward_drive_arm.STL" scale="0.01 0.01 0.01" />
+            </geometry>
+        </collision>
     </link>
     <joint name="joint_2" type="revolute">
@@ -55,4 +73,10 @@
             </geometry>
         </visual>
+        <collision>
+            <origin xyz="-0.03 -0.4 -0.06" rpy="${PI/2} 0 ${PI/2}" />
+            <geometry>
+                <mesh filename="package://zimo_description/meshes/zimo/horizontal_arm.STL" scale="0.01 0.01 0.01" />
+            </geometry>
+        </collision>
     </link>
     <joint name="joint_3" type="revolute">
@@ -70,4 +94,10 @@
             </geometry>
         </visual>
+        <collision>
+            <origin xyz="0 -0.05 -0.15" rpy="0 0 ${PI/2}" />
+            <geometry>
+                <mesh filename="package://zimo_description/meshes/zimo/claw_support.STL" scale="0.01 0.01 0.01" />
+            </geometry>
+        </collision>
     </link>
     <joint name="joint_4" type="fixed">
@@ -83,4 +113,10 @@
             </geometry>
         </visual>
+        <collision>
+            <origin xyz="-0.1 0.5 -0.1" rpy="0 0 -${PI/2}" />
+            <geometry>
+                <mesh filename="package://zimo_description/meshes/zimo/right_finger.STL" scale="0.01 0.01 0.01" />
+            </geometry>
+        </collision>
     </link>
     <joint name="joint_5" type="revolute">
@@ -98,4 +134,10 @@
             </geometry>
         </visual>
+        <collision>
+            <origin xyz="-0.04 0.5 -0.1" rpy="0 0 -${PI/2}" />
+            <geometry>
+                <mesh filename="package://zimo_description/meshes/zimo/left_finger.STL" scale="0.01 0.01 0.01" />
+            </geometry>
+        </collision>
     </link>
     <joint name="joint_6" type="revolute">

Commit message: third commit

File: zimo_description/urdf/zimo.urdf.xacro (robot description, xacro)
@@ -4,6 +4,16 @@
     <xacro:property name="effort" value="30.0" />
     <xacro:property name="velocity" value="10.0" />
+    <!-- Corrected macro definition -->
+    <xacro:macro name="default_inertial" params="mass">
+        <inertial>
+            <mass value="${mass}" />
+            <inertia ixx="1.0" ixy="0.0" ixz="0.0"
+                     iyy="1.0" iyx="0.0"
+                     izz="1.0"/>
+        </inertial>
+    </xacro:macro>
     <link name="world" />
     <link name="base_link">
+        <xacro:default_inertial mass="1.0" />
         <visual>
             <origin xyz="-0.5 -0.5 0" rpy="0 0 0" />
@@ -25,4 +35,5 @@
     </joint>
     <link name="base_plate">
+        <xacro:default_inertial mass="0.1" />
         <visual>
             <origin xyz="-0.39 -0.39 -0.56" rpy="0 0 0" />
@@ -46,4 +57,5 @@
     </joint>
     <link name="forward_drive_arm">
+        <xacro:default_inertial mass="0.1" />
         <visual>
             <origin xyz="0.19 -0.06 -0.08" rpy="0 -${PI/2} ${PI/2}" />
@@ -67,4 +79,5 @@
     </joint>
     <link name="horizontal_arm">
+        <xacro:default_inertial mass="0.1" />
         <visual>
             <origin xyz="-0.03 -0.4 -0.06" rpy="${PI/2} 0 ${PI/2}" />
@@ -88,4 +101,5 @@
     </joint>
     <link name="claw_support">
+        <xacro:default_inertial mass="0.05" />
         <visual>
             <origin xyz="0 -0.05 -0.15" rpy="0 0 ${PI/2}" />
@@ -107,4 +121,5 @@
     </joint>
     <link name="right_grip">
+        <xacro:default_inertial mass="0.01" />
         <visual>
             <origin xyz="-0.1 0.5 -0.1" rpy="0 0 -${PI/2}" />
@@ -128,4 +143,5 @@
     </joint>
     <link name="left_grip">
+        <xacro:default_inertial mass="0.01" />
         <visual>
             <origin xyz="-0.04 0.5 -0.1" rpy="0 0 -${PI/2}" />

Commit message: fifth commit

File: zimo_description/urdf/zimo.urdf.xacro (robot description, xacro)
@@ -2,6 +2,6 @@
 <robot xmlns:xacro="http://www.ros.org/wiki/xacro" name="zimo">
     <xacro:arg name="is_ignition" default="true" />
+    <xacro:include filename="$(find zimo_description)/urdf/zimo_ros2_controller.xacro" />
     <xacro:include filename="$(find zimo_description)/urdf/zimo_gazebo.xacro" />
-    <xacro:include filename="$(find zimo_description)/urdf/zimo_ros2_controller.xacro" />
     <xacro:property name="PI" value="3.14159" />
     <xacro:property name="effort" value="30.0" />

File: zimo_description/urdf/zimo_gazebo.xacro (robot description, xacro)
@@ -1,15 +1,14 @@
 <?xml version="1.0"?>
 <robot xmlns:xacro="http://www.ros.org/wiki/xacro" name="zimo">
+    <xacro:arg name="is_ignition" default="true" />
     <gazebo>
-        <xacro:if value="$(arg is_ignition)">
+        <xacro:if value="${is_ignition}">
             <plugin filename="ign_ros2_control_system" name="ign_ros2_control::IgnitionROS2ControlPlugin">
-                <parameter>
-                </parameter>
+                <parameter>$(find zimo_controller)/config/zimo_controller.yaml</parameter>
             </plugin>
         </xacro:if>
-        <xacro:unless value="$(args is_ignition)">
+        <xacro:unless value="${is_ignition}">
             <plugin filename="gz_ros2_control_system" name="gz_ros2_control::GazeboSimROS2ControlPlugin">
-                <parameter>
-                </parameter>
+                <parameter>$(find zimo_controller)/config/zimo_controller.yaml</parameter>
             </plugin>
         </xacro:unless>

File: zimo_description/urdf/zimo_ros2_controller.xacro (robot description, xacro)
@@ -1,45 +1,47 @@
 <?xml version="1.0"?>
 <robot xmlns:xacro="http://www.ros.org/wiki/xacro" name="zimo">
+    <xacro:arg name="is_ignition" default="true" />
     <xacro:property name="PI" value="3.14159" />
     <ros2_control type="system" name="RobotSystem">
-        <xacro:if value="$(arg is_ignition)">
+        <xacro:if value="${is_ignition}">
             <hardware>
-                <plugin>ign_ros2_control/IgnitiionSystem</plugin>
+                <plugin>ign_ros2_control/IgnitionSystem</plugin>
             </hardware>
         </xacro:if>
-        <xacro:unless value="$(arg is_ignition)">
-            <plugin>gz_ros2_control/GazeboSimSystem</plugin>
+        <xacro:unless value="${is_ignition}">
+            <hardware>
+                <plugin>gz_ros2_control/GazeboSimSystem</plugin>
+            </hardware>
         </xacro:unless>
         <joint name="joint_1">
-            <commmand_interface name="position">
-                <param name="min">-${PI/2}</param>
-                <param name="max">${PI/2}</param>
-            </commmand_interface>
-            <state_interface name="postion" />
+            <command_interface name="position">
+                <param name="min">-${PI}/2</param>
+                <param name="max">${PI}/2</param>
+            </command_interface>
+            <state_interface name="position" />
         </joint>
         <joint name="joint_2">
-            <commmand_interface name="position">
-                <param name="min">-${PI/2}</param>
-                <param name="max">${PI/2}</param>
-            </commmand_interface>
-            <state_interface name="postion" />
+            <command_interface name="position">
+                <param name="min">-${PI}/2</param>
+                <param name="max">${PI}/2</param>
+            </command_interface>
+            <state_interface name="position" />
         </joint>
         <joint name="joint_3">
-            <commmand_interface name="position">
-                <param name="min">-${PI/2}</param>
-                <param name="max">${PI/2}</param>
-            </commmand_interface>
-            <state_interface name="postion" />
+            <command_interface name="position">
+                <param name="min">-${PI}/2</param>
+                <param name="max">${PI}/2</param>
+            </command_interface>
+            <state_interface name="position" />
         </joint>
         <joint name="joint_4">
-            <commmand_interface name="position">
-                <param name="min">-${PI/2}</param>
+            <command_interface name="position">
+                <param name="min">-${PI}/2</param>
                 <param name="max">0.0</param>
-            </commmand_interface>
-            <state_interface name="postion" />
+            </command_interface>
+            <state_interface name="position" />
         </joint>
         <joint name="joint_5">
-           <param name="mimic">joint_4</param>
-           <param name="multiplier">-1</param>
+            <mimic joint="joint_4" multiplier="-1" />
         </joint>
     </ros2_control>
